Commit message: feat(v0.3.13)

File: hex_zmq_servers/robot/hexarm/urdf/archer_d6y/empty.urdf (robot description, URDF)
Before this commit: robot archer_y6, 7 links, 6 joints
Links:
- link base_link: mass 0.748 -> 0.687; geometry collision mesh filename=package://xpkg_urdf_archer_d6y/meshes/base_link.STL; visual mesh filename=package://xpkg_urdf_archer_d6y/meshes/base_link.STL
- link link_1: mass 0.2289 -> 0.2154; geometry collision mesh filename=package://xpkg_urdf_archer_d6y/meshes/link_1.STL; visual mesh filename=package://xpkg_urdf_archer_d6y/meshes/link_1.STL
- link link_2: mass 1.5141 -> 1.3123; geometry collision mesh filename=package://xpkg_urdf_archer_d6y/meshes/link_2.STL; visual mesh filename=package://xpkg_urdf_archer_d6y/meshes/link_2.STL
- link link_3: mass 1.2023 -> 1.1083; geometry collision mesh filename=package://xpkg_urdf_archer_d6y/meshes/link_3.STL; visual mesh filename=package://xpkg_urdf_archer_d6y/meshes/link_3.STL
- link link_4: mass 0.6233 -> 0.5398; geometry collision mesh filename=package://xpkg_urdf_archer_d6y/meshes/link_4.STL; visual mesh filename=package://xpkg_urdf_archer_d6y/meshes/link_4.STL
- link link_5: mass 0.4173 -> 0.3984; geometry collision mesh filename=package://xpkg_urdf_archer_d6y/meshes/link_5.STL; visual mesh filename=package://xpkg_urdf_archer_d6y/meshes/link_5.STL
- link link_6: mass 0.7201 -> 0.001; geometry collision mesh filename=package://xpkg_urdf_archer_d6y/meshes/link_6.STL; visual mesh filename=package://xpkg_urdf_archer_d6y/meshes/link_6.STL
Joints:
- joint joint_1: limit lower=-2.91 upper=2.91 effort=6 velocity=6 -> lower=-2.61 upper=3.14 effort=6 velocity=6; origin xyz=0 0 0.06655 rpy=0 0 0 -> xyz=0 0 0.0665 rpy=0 0 0
- joint joint_5: origin xyz=-0.0553 0 0.0702 rpy=0 0 0 -> xyz=-0.0553 0 0.070 rpy=0 0 0
- joint joint_6: origin xyz=0.0552 0 0.02895 rpy=0 0 0 -> xyz=0.0553 0 0.029 rpy=0 0 0

File: hex_zmq_servers/robot/hexarm/urdf/archer_d6y/gp100.urdf (robot description, URDF)
Before this commit: robot archer_y6, 7 links, 6 joints
Links:
- link base_link: mass 0.748 -> 0.687; geometry collision mesh filename=package://xpkg_urdf_archer_d6y/meshes/base_link.STL; visual mesh filename=package://xpkg_urdf_archer_d6y/meshes/base_link.STL
- link link_1: mass 0.2289 -> 0.2154; geometry collision mesh filename=package://xpkg_urdf_archer_d6y/meshes/link_1.STL; visual mesh filename=package://xpkg_urdf_archer_d6y/meshes/link_1.STL
- link link_2: mass 1.5141 -> 1.3123; geometry collision mesh filename=package://xpkg_urdf_archer_d6y/meshes/link_2.STL; visual mesh filename=package://xpkg_urdf_archer_d6y/meshes/link_2.STL
- link link_3: mass 1.2023 -> 1.1083; geometry collision mesh filename=package://xpkg_urdf_archer_d6y/meshes/link_3.STL; visual mesh filename=package://xpkg_urdf_archer_d6y/meshes/link_3.STL
- link link_4: mass 0.6233 -> 0.5398; geometry collision mesh filename=package://xpkg_urdf_archer_d6y/meshes/link_4.STL; visual mesh filename=package://xpkg_urdf_archer_d6y/meshes/link_4.STL
- link link_5: mass 0.4173 -> 0.3984; geometry collision mesh filename=package://xpkg_urdf_archer_d6y/meshes/link_5.STL; visual mesh filename=package://xpkg_urdf_archer_d6y/meshes/link_5.STL
- link link_6: mass 0.7201 -> 0.6760; geometry collision mesh filename=package://xpkg_urdf_archer_d6y/meshes/link_6.STL; visual mesh filename=package://xpkg_urdf_archer_d6y/meshes/link_6.STL
Joints:
- joint joint_1: limit lower=-2.91 upper=2.91 effort=6 velocity=6 -> lower=-2.61 upper=3.14 effort=6 velocity=6; origin xyz=0 0 0.06655 rpy=0 0 0 -> xyz=0 0 0.0665 rpy=0 0 0
- joint joint_5: origin xyz=-0.0553 0 0.0702 rpy=0 0 0 -> xyz=-0.0553 0 0.070 rpy=0 0 0
- joint joint_6: origin xyz=0.0552 0 0.02895 rpy=0 0 0 -> xyz=0.0553 0 0.029 rpy=0 0 0

File: hex_zmq_servers/robot/hexarm/urdf/archer_d6y/gp100_handle.urdf (robot description, URDF)
Before this commit: robot archer_y6, 7 links, 6 joints
Links:
- link base_link: mass 0.748 -> 0.687; geometry collision mesh filename=package://xpkg_urdf_archer_d6y/meshes/base_link.STL; visual mesh filename=package://xpkg_urdf_archer_d6y/meshes/base_link.STL
- link link_1: mass 0.2289 -> 0.2154; geometry collision mesh filename=package://xpkg_urdf_archer_d6y/meshes/link_1.STL; visual mesh filename=package://xpkg_urdf_archer_d6y/meshes/link_1.STL
- link link_2: mass 1.5141 -> 1.3123; geometry collision mesh filename=package://xpkg_urdf_archer_d6y/meshes/link_2.STL; visual mesh filename=package://xpkg_urdf_archer_d6y/meshes/link_2.STL
- link link_3: mass 1.2023 -> 1.1083; geometry collision mesh filename=package://xpkg_urdf_archer_d6y/meshes/link_3.STL; visual mesh filename=package://xpkg_urdf_archer_d6y/meshes/link_3.STL
- link link_4: mass 0.6233 -> 0.5398; geometry collision mesh filename=package://xpkg_urdf_archer_d6y/meshes/link_4.STL; visual mesh filename=package://xpkg_urdf_archer_d6y/meshes/link_4.STL
- link link_5: mass 0.4173 -> 0.3984; geometry collision mesh filename=package://xpkg_urdf_archer_d6y/meshes/link_5.STL; visual mesh filename=package://xpkg_urdf_archer_d6y/meshes/link_5.STL
- link link_6: geometry collision mesh filename=package://xpkg_urdf_archer_d6y/meshes/link_6.STL; visual mesh filename=package://xpkg_urdf_archer_d6y/meshes/link_6.STL
Joints:
- joint joint_1: limit lower=-2.91 upper=2.91 effort=6 velocity=6 -> lower=-2.61 upper=3.14 effort=6 velocity=6; origin xyz=0 0 0.06655 rpy=0 0 0 -> xyz=0 0 0.0665 rpy=0 0 0
- joint joint_5: origin xyz=-0.0553 0 0.0702 rpy=0 0 0 -> xyz=-0.0553 0 0.070 rpy=0 0 0
- joint joint_6: origin xyz=0.0552 0 0.02895 rpy=0 0 0 -> xyz=0.0553 0 0.029 rpy=0 0 0

File: hex_zmq_servers/robot/hexarm/urdf/archer_d6y/gp100_p050.urdf (robot description, URDF)
Before this commit: robot archer_y6, 7 links, 6 joints
Links:
- link base_link: mass 0.748 -> 0.687; geometry collision mesh filename=package://xpkg_urdf_archer_d6y/meshes/base_link.STL; visual mesh filename=package://xpkg_urdf_archer_d6y/meshes/base_link.STL
- link link_1: mass 0.2289 -> 0.2154; geometry collision mesh filename=package://xpkg_urdf_archer_d6y/meshes/link_1.STL; visual mesh filename=package://xpkg_urdf_archer_d6y/meshes/link_1.STL
- link link_2: mass 1.5141 -> 1.3123; geometry collision mesh filename=package://xpkg_urdf_archer_d6y/meshes/link_2.STL; visual mesh filename=package://xpkg_urdf_archer_d6y/meshes/link_2.STL
- link link_3: mass 1.2023 -> 1.1083; geometry collision mesh filename=package://xpkg_urdf_archer_d6y/meshes/link_3.STL; visual mesh filename=package://xpkg_urdf_archer_d6y/meshes/link_3.STL
- link link_4: mass 0.6233 -> 0.5398; geometry collision mesh filename=package://xpkg_urdf_archer_d6y/meshes/link_4.STL; visual mesh filename=package://xpkg_urdf_archer_d6y/meshes/link_4.STL
- link link_5: mass 0.4173 -> 0.3984; geometry collision mesh filename=package://xpkg_urdf_archer_d6y/meshes/link_5.STL; visual mesh filename=package://xpkg_urdf_archer_d6y/meshes/link_5.STL
- link link_6: mass 0.7201 -> 0.7751; geometry collision mesh filename=package://xpkg_urdf_archer_d6y/meshes/link_6.STL; visual mesh filename=package://xpkg_urdf_archer_d6y/meshes/link_6.STL
Joints:
- joint joint_1: limit lower=-2.91 upper=2.91 effort=6 velocity=6 -> lower=-2.61 upper=3.14 effort=6 velocity=6; origin xyz=0 0 0.06655 rpy=0 0 0 -> xyz=0 0 0.0665 rpy=0 0 0
- joint joint_5: origin xyz=-0.0553 0 0.0702 rpy=0 0 0 -> xyz=-0.0553 0 0.070 rpy=0 0 0
- joint joint_6: origin xyz=0.0552 0 0.02895 rpy=0 0 0 -> xyz=0.0553 0 0.029 rpy=0 0 0

File: hex_zmq_servers/robot/hexarm/urdf/archer_d6y/gp100_p050_handle.urdf (robot description, URDF)
Before this commit: robot archer_y6, 7 links, 6 joints
Links:
- link base_link: mass 0.748 -> 0.687; geometry collision mesh filename=package://xpkg_urdf_archer_d6y/meshes/base_link.STL; visual mesh filename=package://xpkg_urdf_archer_d6y/meshes/base_link.STL
- link link_1: mass 0.2289 -> 0.2154; geometry collision mesh filename=package://xpkg_urdf_archer_d6y/meshes/link_1.STL; visual mesh filename=package://xpkg_urdf_archer_d6y/meshes/link_1.STL
- link link_2: mass 1.5141 -> 1.3123; geometry collision mesh filename=package://xpkg_urdf_archer_d6y/meshes/link_2.STL; visual mesh filename=package://xpkg_urdf_archer_d6y/meshes/link_2.STL
- link link_3: mass 1.2023 -> 1.1083; geometry collision mesh filename=package://xpkg_urdf_archer_d6y/meshes/link_3.STL; visual mesh filename=package://xpkg_urdf_archer_d6y/meshes/link_3.STL
- link link_4: mass 0.6233 -> 0.5398; geometry collision mesh filename=package://xpkg_urdf_archer_d6y/meshes/link_4.STL; visual mesh filename=package://xpkg_urdf_archer_d6y/meshes/link_4.STL
- link link_5: mass 0.4173 -> 0.3984; geometry collision mesh filename=package://xpkg_urdf_archer_d6y/meshes/link_5.STL; visual mesh filename=package://xpkg_urdf_archer_d6y/meshes/link_5.STL
- link link_6: mass 0.7201 -> 0.8192; geometry collision mesh filename=package://xpkg_urdf_archer_d6y/meshes/link_6.STL; visual mesh filename=package://xpkg_urdf_archer_d6y/meshes/link_6.STL
Joints:
- joint joint_1: limit lower=-2.91 upper=2.91 effort=6 velocity=6 -> lower=-2.61 upper=3.14 effort=6 velocity=6; origin xyz=0 0 0.06655 rpy=0 0 0 -> xyz=0 0 0.0665 rpy=0 0 0
- joint joint_5: origin xyz=-0.0553 0 0.0702 rpy=0 0 0 -> xyz=-0.0553 0 0.070 rpy=0 0 0
- joint joint_6: origin xyz=0.0552 0 0.02895 rpy=0 0 0 -> xyz=0.0553 0 0.029 rpy=0 0 0

File: hex_zmq_servers/robot/hexarm/urdf/archer_y6/empty.urdf (robot description, URDF)
Before this commit: robot archer_y6, 7 links, 6 joints
Links:
- link base_link: mass 0.687 -> 0.748
- link link_1: mass 0.2154 -> 0.2289
- link link_2: mass 1.3123 -> 1.5141
- link link_3: mass 1.1083 -> 1.2023
- link link_4: mass 0.5398 -> 0.6233
- link link_5: mass 0.3984 -> 0.4173
Joints:
- joint joint_1: limit lower=-2.61 upper=3.14 effort=6 velocity=6 -> lower=-2.91 upper=2.91 effort=6 velocity=6; origin xyz=0 0 0.0665 rpy=0 0 0 -> xyz=0 0 0.06655 rpy=0 0 0
- joint joint_5: origin xyz=-0.0553 0 0.070 rpy=0 0 0 -> xyz=-0.0553 0 0.0702 rpy=0 0 0
- joint joint_6: origin xyz=0.0553 0 0.029 rpy=0 0 0 -> xyz=0.0552 0 0.02895 rpy=0 0 0

File: hex_zmq_servers/robot/hexarm/urdf/archer_y6/gp100.urdf (robot description, URDF)
Before this commit: robot archer_y6, 7 links, 6 joints
Links:
- link base_link: mass 0.687 -> 0.748
- link link_1: mass 0.2154 -> 0.2289
- link link_2: mass 1.3123 -> 1.5141
- link link_3: mass 1.1083 -> 1.2023
- link link_4: mass 0.5398 -> 0.6233
- link link_5: mass 0.3984 -> 0.4173
Joints:
- joint joint_1: limit lower=-2.61 upper=3.14 effort=6 velocity=6 -> lower=-2.91 upper=2.91 effort=6 velocity=6; origin xyz=0 0 0.0665 rpy=0 0 0 -> xyz=0 0 0.06655 rpy=0 0 0
- joint joint_5: origin xyz=-0.0553 0 0.070 rpy=0 0 0 -> xyz=-0.0553 0 0.0702 rpy=0 0 0
- joint joint_6: origin xyz=0.0553 0 0.029 rpy=0 0 0 -> xyz=0.0552 0 0.02895 rpy=0 0 0

File: hex_zmq_servers/robot/hexarm/urdf/archer_y6/gp100_p050.urdf (robot description, URDF)
Before this commit: robot archer_y6, 7 links, 6 joints
Links:
- link base_link: mass 0.687 -> 0.748
- link link_1: mass 0.2154 -> 0.2289
- link link_2: mass 1.3123 -> 1.5141
- link link_3: mass 1.1083 -> 1.2023
- link link_4: mass 0.5398 -> 0.6233
- link link_5: mass 0.3984 -> 0.4173
Joints:
- joint joint_1: limit lower=-2.61 upper=3.14 effort=6 velocity=6 -> lower=-2.91 upper=2.91 effort=6 velocity=6; origin xyz=0 0 0.0665 rpy=0 0 0 -> xyz=0 0 0.06655 rpy=0 0 0
- joint joint_5: origin xyz=-0.0553 0 0.070 rpy=0 0 0 -> xyz=-0.0553 0 0.0702 rpy=0 0 0
- joint joint_6: origin xyz=0.0553 0 0.029 rpy=0 0 0 -> xyz=0.0552 0 0.02895 rpy=0 0 0

File: hex_zmq_servers/robot/hexarm/urdf/archer_y6/gp100_p050_handle.urdf (robot description, URDF)
Before this commit: robot archer_y6, 7 links, 6 joints
Links:
- link base_link: mass 0.687 -> 0.748
- link link_1: mass 0.2154 -> 0.2289
- link link_2: mass 1.3123 -> 1.5141
- link link_3: mass 1.1083 -> 1.2023
- link link_4: mass 0.5398 -> 0.6233
- link link_5: mass 0.3984 -> 0.4173
Joints:
- joint joint_1: limit lower=-2.61 upper=3.14 effort=6 velocity=6 -> lower=-2.91 upper=2.91 effort=6 velocity=6; origin xyz=0 0 0.0665 rpy=0 0 0 -> xyz=0 0 0.06655 rpy=0 0 0
- joint joint_5: origin xyz=-0.0553 0 0.070 rpy=0 0 0 -> xyz=-0.0553 0 0.0702 rpy=0 0 0
- joint joint_6: origin xyz=0.0553 0 0.029 rpy=0 0 0 -> xyz=0.0552 0 0.02895 rpy=0 0 0
