Commit message: feat: add MuJoCo simulation support for archer_l6y
- Add mujoco_archer_l6y example and config
- Add L6Y MuJoCo model (archer_l6y/)
- Add l6y_gp100.urdf with gripper
- Add xpkg_urdf source files for archer_l6y and gp100
- Update cam/mujoco/robot modules for better integration

File: hex_zmq_servers/robot/hexarm/urdf/archer_l6y/gp100_d435i.urdf (robot description, URDF)
Before this commit: robot archer_l6y, 7 links, 6 joints
Joints:
- joint joint_4: origin xyz=-0.065 -5E-05 0.25 rpy=0 0 0 -> xyz=-0.065 0 0.25 rpy=0 0 0
