Commit message: update gripper close position

File: hex_zmq_servers/robot/hexarm/urdf/firefly_y6/y6_gr100.urdf (robot description, URDF)
Before this commit: robot firefly_y6_gr100, 11 links, 10 joints
Joints:
- joint gripper_left_joint_1: limit lower=0.0 upper=0.57 effort=5 velocity=10 -> lower=0.0 upper=0.9 effort=5 velocity=10
- joint gripper_right_joint_1: limit lower=0.0 upper=0.57 effort=5 velocity=10 -> lower=0.0 upper=0.9 effort=5 velocity=10
