Commit message: firefly_y6: swap GR100 for Tianyi 总装 gripper
New gripper meshes (Link_1/2/3 -> gripper_base_link/L1/L2). MJCF gripper subtree:
mount at link_6 (Rz+90 to match the soda-ui render), two claws axis 0 0 -1 with
right mimicking left (equality polycoef -1) + contact excludes. URDF: gr100.urdf
link_6 lumped mass 0.535->0.325 kg; y6_gr100.urdf gripper joints/origins/mimic.
Wrist camera + 0.187 TCP unchanged.

File: hex_zmq_servers/robot/hexarm/urdf/firefly_y6/gr100.urdf (robot description, URDF)
Before this commit: robot firefly_y6, 7 links, 6 joints
Links:
- link link_6: mass 0.5354 -> 0.32481

File: hex_zmq_servers/robot/hexarm/urdf/firefly_y6/y6_gr100.urdf (robot description, URDF)
Before this commit: robot firefly_y6_gr100, 11 links, 10 joints
Joints:
- joint gripper_base_joint: origin xyz=0 0 0 rpy=0 0 0 -> xyz=0 0 0 rpy=0 0 -1.5707963
- joint gripper_left_joint_1: axis -1 0 0 -> 0 0 1; origin xyz=0 -0.015 0.076799 rpy=0 0 0 -> xyz=-0.015 0.01475 0.07679888 rpy=0 1.57079633 -1.57079633
- joint gripper_right_joint_1: axis 1 0 0 -> 0 0 1; limit lower=0.0 upper=0.9 effort=5 velocity=10 -> lower=-0.9 upper=0.9 effort=5 velocity=10; mimic joint=gripper_left_joint_1 multiplier=1.0 offset=0 -> joint=gripper_left_joint_1 multiplier=-1.0 offset=0; origin xyz=0 0.015 0.076799 rpy=0 0 0 -> xyz=0.015 0.01475 0.07679888 rpy=0 1.57079633 -1.57079633

Commit message: rotate teleop axis

File: hex_zmq_servers/robot/hexarm/urdf/firefly_y6/gr100.urdf (robot description, URDF)
Before this commit: robot firefly_y6, 7 links, 6 joints
Links:
- link link_6: mass 0.32481 -> 0.5354
